Commit message: update drive_bot.cpp, update my_robot.xacro

File: src/my_robot/urdf/my_robot.xacro (robot description, xacro)
@@ -1,4 +1,5 @@
 <?xml version='1.0'?>
 <robot name="my_robot" xmlns:xacro="http://www.ros.org/wiki/xacro">
+  <xacro:include filename="$(find my_robot)/urdf/my_robot.gazebo" />
   <link name="robot_footprint"></link>
   <joint name="robot_footprint_joint" type="fixed">
@@ -11,5 +12,5 @@
     <inertial>
       <mass value="15.0"/>
-      <origin xyz="0.0 0 0" rpy=" 0 0 0"/>
+      <origin xyz="0 0 0" rpy="0 0 0"/>
       <inertia
           ixx="0.1" ixy="0" ixz="0"
@@ -25,5 +26,5 @@
     </collision>
     <visual name='chassis_visual'>
-      <origin xyz="0 0 0" rpy=" 0 0 0"/>
+      <origin xyz="0 0 0" rpy="0 0 0"/>
       <geometry>
         <box size=".4 .2 .1"/>
@@ -31,5 +32,5 @@
     </visual>
     <collision name='back_caster_collision'>
-      <origin xyz="-0.15 0 -0.05" rpy=" 0 0 0"/>
+      <origin xyz="-0.15 0 -0.05" rpy="0 0 0"/>
       <geometry>
         <sphere radius="0.0499"/>
@@ -37,5 +38,5 @@
     </collision>
     <visual name='back_caster_visual'>
-      <origin xyz="-0.15 0 -0.05" rpy=" 0 0 0"/>
+      <origin xyz="-0.15 0 -0.05" rpy="0 0 0"/>
       <geometry>
         <sphere radius="0.05"/>
@@ -43,5 +44,5 @@
     </visual>
     <collision name='front_caster_collision'>
-      <origin xyz="0.15 0 -0.05" rpy=" 0 0 0"/>
+      <origin xyz="0.15 0 -0.05" rpy="0 0 0"/>
       <geometry>
         <sphere radius="0.0499"/>
@@ -49,5 +50,5 @@
     </collision>
     <visual name='front_caster_visual'>
-      <origin xyz="0.15 0 -0.05" rpy=" 0 0 0"/>
+      <origin xyz="0.15 0 -0.05" rpy="0 0 0"/>
       <geometry>
         <sphere radius="0.05"/>
@@ -122,5 +123,5 @@
     <inertial>
       <mass value="0.1"/>
-      <origin xyz="0 0 0" rpy=" 0 0 0"/>
+      <origin xyz="0 0 0" rpy="0 0 0"/>
       <inertia
           ixx="1e-6" ixy="0" ixz="0"
@@ -130,5 +131,5 @@
     </inertial>
     <collision name='camera_collision'>
-      <origin xyz="0 0 0" rpy=" 0 0 0"/>
+      <origin xyz="0 0 0" rpy="0 0 0"/>
       <geometry>
         <box size="0 0 0"/>
@@ -153,5 +154,5 @@
     <inertial>
       <mass value="1e-5"/>
-      <origin xyz="0 0 0" rpy=" 0 0 0"/>
+      <origin xyz="0 0 0" rpy="0 0 0"/>
       <inertia
           ixx="1e-6" ixy="0" ixz="0"
@@ -161,5 +162,5 @@
     </inertial>
     <collision name='hokuyo_collision'>
-      <origin xyz="0 0 0" rpy=" 0 0 0"/>
+      <origin xyz="0 0 0" rpy="0 0 0"/>
       <geometry>
         <box size="0.1 0.1 0.1"/>
