Commit message: Update ball_chaser

File: my_robot/urdf/my_robot.xacro (robot description, xacro)
@@ -22,5 +22,5 @@
       <origin xyz="0 0 0" rpy="0 0 0"/>
       <geometry>
-        <box size=".5 .4 .1"/>
+        <box size=".6 .4 .1"/>
       </geometry>
     </collision>
@@ -28,9 +28,9 @@
       <origin xyz="0 0 0" rpy="0 0 0"/>
       <geometry>
-        <box size=".5 .4 .1"/>
+        <box size=".6 .4 .1"/>
       </geometry>
     </visual>
     <collision name='back_caster_collision'>
-      <origin xyz="-0.13 0 -0.05" rpy="0 0 0"/>
+      <origin xyz="-0.15 0 -0.05" rpy="0 0 0"/>
       <geometry>
         <sphere radius="0.0499"/>

Commit message: project2 submission

File: my_robot/urdf/my_robot.xacro (robot description, xacro)
@@ -30,4 +30,7 @@
         <box size=".6 .4 .1"/>
       </geometry>
+      <material name='chassis_color'>
+  	<color rgba="0.3 .5 0.3 0.3"/>
+      </material>
     </visual>
     <collision name='back_caster_collision'>
