Commit message: amend myworld.world

File: my_robot/urdf/cam_robot.xacro (robot description, xacro)
@@ -1,5 +1,5 @@
 <?xml version="1.0"?>
-<robot name="my_robot" xmlns:xacro="http://www.ros.org/wiki/xacro">
-  <xacro:include filename="$(find my_robot)/urdf/my_robot.gazebo"/>
+<robot name="cam_robot" xmlns:xacro="http://www.ros.org/wiki/xacro">
+  <xacro:include filename="$(find my_robot)/urdf/cam_robot.gazebo"/>
   <link name="robot_footprint"></link>
   <joint name="robot_footprint_joint" type="fixed">
@@ -37,5 +37,5 @@
       <origin xyz="-0.15 0 -0.05" rpy="0 0 0"/>
       <geometry>
-        <sphere radius="0.0499"/>
+        <sphere radius="0.05"/>
       </geometry>
     </collision>
@@ -49,5 +49,5 @@
       <origin xyz="0.15 0 -0.05" rpy="0 0 0"/>
       <geometry>
-        <sphere radius="0.0499"/>
+        <sphere radius="0.05"/>
       </geometry>
     </collision>

Commit message: change process_images

File: my_robot/urdf/cam_robot.xacro (robot description, xacro)
@@ -9,5 +9,4 @@
   </joint>
   <link name='chassis'>
-    <pose>0 0 0.1 0 0 0</pose>
     <inertial>
     <mass value="20.0"/>
@@ -22,5 +21,5 @@
       <origin xyz="0 0 0" rpy="0 0 0"/>
       <geometry>
-        <box size=".6 .4 .1"/>
+        <box size=".6 .4 .2"/>
       </geometry>
     </collision>
@@ -28,8 +27,8 @@
       <origin xyz="0 0 0" rpy="0 0 0"/>
       <geometry>
-        <box size=".6 .4 .1"/>
+        <box size=".6 .4 .2"/>
       </geometry>
       <material name='chassis_color'>
-  	<color rgba="0.3 .5 0.3 0.3"/>
+  	<color rgba="0 0 0.8 1"/>
       </material>
     </visual>
@@ -37,5 +36,5 @@
       <origin xyz="-0.15 0 -0.05" rpy="0 0 0"/>
       <geometry>
-        <sphere radius="0.05"/>
+        <sphere radius="0.1"/>
       </geometry>
     </collision>
@@ -43,5 +42,5 @@
       <origin xyz="-0.15 0 -0.05" rpy="0 0 0"/>
       <geometry>
-        <sphere radius="0.05"/>
+        <sphere radius="0.1"/>
       </geometry>
     </visual>
@@ -49,5 +48,5 @@
       <origin xyz="0.15 0 -0.05" rpy="0 0 0"/>
       <geometry>
-        <sphere radius="0.05"/>
+        <sphere radius="0.1"/>
       </geometry>
     </collision>
@@ -55,13 +54,12 @@
       <origin xyz="0.15 0 -0.05" rpy="0 0 0"/>
       <geometry>
-        <sphere radius="0.05"/>
+        <sphere radius="0.1"/>
       </geometry>
     </visual>
   </link>
   <link name="left_wheel">
-    <pose>0 0 0.1 0 0 0</pose>
     <inertial>
       <mass value="5"/>
-      <origin xyz="0 0 0" rpy="0 1.5707 1.5707"/>
+      <origin xyz="0 0.2 0.2" rpy="0 1.5707 1.5707"/>
       <inertia
         ixx="0.1" ixy="0" ixz="0"
@@ -71,21 +69,20 @@
     </inertial>
     <visual name="left_wheel_visual">
-      <origin xyz="0 0 0" rpy="0 1.5707 1.5707"/>
+      <origin xyz="0 0.05 0" rpy="0 1.5707 1.5707"/>
       <geometry>
-        <cylinder radius="0.3" length="0.05"/>
+        <cylinder radius="0.15" length="0.05"/>
       </geometry>
     </visual>
     <collision name="left_wheel_collision">
-      <origin xyz="0 0 0" rpy="0 1.5707 1.5707"/>
+      <origin xyz="0 0.05 0" rpy="0 1.5707 1.5707"/>
       <geometry>
-        <cylinder radius="0.3" length="0.05"/>
+        <cylinder radius="0.15" length="0.05"/>
       </geometry>
     </collision>
   </link>
   <link name="right_wheel">
-    <pose>0 0 -0.1 0 0 0</pose>
     <inertial>
       <mass value="5"/>
-      <origin xyz="0 0 0" rpy="0 1.5707 1.5707"/>
+      <origin xyz="0 -0.2 0.2" rpy="0 1.5707 1.5707"/>
       <inertia
         ixx="0.1" ixy="0" ixz="0"
@@ -95,18 +92,18 @@
     </inertial>
     <visual name="right_wheel_visual">
-      <origin xyz="0 0 0" rpy="0 1.5707 1.5707"/>
+      <origin xyz="0 -0.05 0" rpy="0 1.5707 1.5707"/>
       <geometry>
-        <cylinder radius="0.3" length="0.05"/>
+        <cylinder radius="0.15" length="0.05"/>
       </geometry>
     </visual>
     <collision name="right_wheel_collision">
-      <orgin xyz="0 0 0 " rpy="0 1.5707 1.5707"/>
+      <orgin xyz="0 -0.05 0" rpy="0 1.5707 1.5707"/>
       <geometry>
-        <cylinder radius="0.3" length="0.05"/>
+        <cylinder radius="0.15" length="0.05"/>
       </geometry>
     </collision>
   </link>
   <joint type="continuous" name="left_wheel_hinge">
-    <origin xyz="0 0.15 0" rpy="0 0 0"/>
+    <origin xyz="0 0.2 0"/>
     <child link="left_wheel"/>
     <parent link="chassis"/>
@@ -116,5 +113,5 @@
   </joint>
   <joint type="continuous" name="right_wheel_hinge">
-    <origin xyz="0 -0.15 0" rpy="0 0 0"/>
+    <origin xyz="0 -0.2 0"/>
     <child link="right_wheel"/>
     <parent link="chassis"/>
@@ -126,5 +123,5 @@
     <inertial>
       <mass value="0.1"/>
-      <origin xyz="0 0 0" rpy="0 0 0"/>
+      <origin xyz="0.3 0 0" rpy="0 0 0"/>
       <inertia
         ixx="1e-6" ixy="0" ixz="0"
@@ -136,5 +133,5 @@
       <origin xyz="0 0 0" rpy="0 0 0"/>
       <geometry>
-        <box size="0.1 0.1 0.1"/>
+        <box size="0.05 0.05 0.05"/>
       </geometry>
       <box_inertia m="0.1" x="0.05" y="0.05" z="0.05"/>
@@ -149,5 +146,5 @@
   </link>
   <joint type="fixed" name="camera_joint">
-    <origin xyz="0.2 0 0" rpy="0 0 0"/>
+    <origin xyz="0.3 0 0" rpy="0 0 0"/>
     <child link="camera"/>
     <parent link="chassis"/>
@@ -178,5 +175,5 @@
   </link>
   <joint type="fixed" name="hokuyo_joint">
-    <origin xyz="0.15 0 0.1" rpy="0 0 0"/>
+    <origin xyz="0.2 0 0.1" rpy="0 0 0"/>
     <child link="hokuyo"/>
     <parent link="chassis"/>
